Commit message: SDF generation, startmove.py test script, new world file. Tweaks to inertia to try to make the damn thing go up steps.

File: defs/jcf.xacro (robot description, xacro)
@@ -148,6 +148,6 @@
       <mass value="0.1"/>
       <origin xyz="0 0 0"/>
-      <inertia ixx="0.012411765597" ixy="-0.000711733678" ixz="0.00050272983"
-        iyy="0.015218160428" iyz="-0.000004273467" izz="0.011763977943"/>
+      <inertia ixx="0.12411765597" ixy="-0.00711733678" ixz="0.0050272983"
+        iyy="0.15218160428" iyz="-0.00004273467" izz="0.11763977943"/>
     </inertial>
     <visual name="pioneer_geom">
@@ -246,17 +246,17 @@
     <link name="${side}_wheel">
       <inertial>
-        <mass value="0.01"/>
-        <origin xyz="0 0 0"/>
+        <mass value="10"/>
+        <origin xyz="0 0 0" rpy="0 1 0"/>
         <inertia
-          ixx="0.000165935"
+          ixx="0.165935"
           ixy="0"
           ixz="0"
-          iyy="0.000317959"
+          iyy="0.317959"
           iyz="0"
-          izz="0.000165935"
+          izz="0.165935"
         />
       </inertial>
       <visual>
-        <origin xyz="0 0 0" rpy="0 0 0"/>
+        <origin xyz="0 0 0" rpy="0 1 0"/>
         <geometry>
           <mesh filename="package://gazebo_ros_3dx/meshes/p3dx_meshes/${side}_wheel.stl"/>
@@ -275,4 +275,6 @@
     <gazebo reference="${side}_wheel">
       <material value="Gazebo/Black"/>
+      <mu1>10</mu1> <!-- rubber friction coeff. -->
+      <mu2>10</mu2>
     </gazebo>
     <joint name="${side}_wheel_joint" type="continuous">

Commit message: sonars positioned (front)

File: defs/jcf.xacro (robot description, xacro)
@@ -5,4 +5,5 @@
   xmlns:xacro="http://ros.org/wiki/xacro"
   name="pioneer3dx">
+  <xacro:include filename="$(find gazebo_ros_3dx)/defs/sonar_sensor.urdf.xacro"/>
   <link name="base_link">
     <!-- The base visual is fine. Just the inertial is questionable.-->
@@ -107,32 +108,4 @@
   </gazebo>
   <!-- Center Wheel + Hubcap -->
-  <!--
-  <link name="center_hubcap">
-    <inertial>
-      <mass value="0.01"/>
-      <origin xyz="0 0 0"/>
-      <inertia ixx="0.012411765597" ixy="-0.000711733678" ixz="0.00050272983"
-        iyy="0.015218160428" iyz="-0.000004273467" izz="0.011763977943"/>
-    </inertial>
-    <visual name="pioneer_geom">
-      <origin xyz="0 0 0" rpy="0 0 0"/>
-      <geometry name="pioneer_geom">
-        <mesh filename="package://gazebo_ros_3dx/meshes/p3dx_meshes/center_hubcap.stl"/>
-      </geometry>
-      <material name="swivel">
-        <color rgba="0.5 0.5 0.5 1"/>
-      </material>
-    </visual>
-    <collision>
-      <origin xyz="0 0 0" rpy="0 0 0"/>
-      <geometry>
-        <box size="0.05 0.05 0.05"/>
-      </geometry>
-    </collision>
-  </link>
-  <gazebo reference="center_hubcap">
-    <material value="Gazebo/Green"/>
-  </gazebo>
-  -->
   <joint name="swivel_hubcap_joint" type="continuous">
     <origin xyz="-0.026 0 -0.016" rpy="0 0 0"/>
@@ -171,11 +144,11 @@
     <material value="Gazebo/Blue"/>
   </gazebo>
-<!--
-  <joint name="center_wheel_joint" type="fixed">
-    <origin xyz="-0.0035 0 -0.001" rpy="0 0 0"/>
-    <parent link="center_wheel"/>
-    <child link="center_hubcap"/>
-  </joint>
--->
+  <!--
+      <joint name="center_wheel_joint" type="fixed">
+        <origin xyz="-0.0035 0 -0.001" rpy="0 0 0"/>
+        <parent link="center_wheel"/>
+        <child link="center_hubcap"/>
+      </joint>
+      -->
   <!-- Front + Back Sonar -->
   <link name="front_sonar">
@@ -229,5 +202,5 @@
       <origin xyz="0 0 0" rpy="0 0 0"/>
       <geometry>
-        <box size=" 0.5 0.25 0.05"/>
+        <box size=" 0 0 0"/>
       </geometry>
     </collision>
@@ -305,20 +278,28 @@
     </plugin>
   </gazebo>
+<!-- test sonar
+  <xacro:sonar_sensor name="s1" parent="base_link"
+    ros_topic="s1" update_rate="10" min_range="0.1" max_range="10"
+    field_of_view="0.267" ray_count="1">
+    <origin xyz="0.2 0 0.22" rpy="0 0 0"/>
+  </xacro:sonar_sensor>
+-->
+  <xacro:include filename="$(find gazebo_ros_3dx)/defs/sonar_pos.urdf.xacro"/>
   <!-- controller
-  <gazebo>
-    <plugin name="differential_drive_controller" filename="libgazebo_ros_diff_drive.so">
-      <updateRate>100.0</updateRate>
-      <robotNamespace>/</robotNamespace>
-      <leftJoint>left_wheel_joint</leftJoint>
-      <rightJoint>right_wheel_joint</rightJoint>
-      <wheelSeparation>0.3</wheelSeparation>
-      <wheelDiameter>0.1</wheelDiameter>
-      <robotBaseFrame>base_link</robotBaseFrame>
-      <torque>200</torque>
-      <commandTopic>cmd_vel</commandTopic>
-      <odometryTopic>odom</odometryTopic>
-      <odometryFrame>odom</odometryFrame>
-    </plugin>
-  </gazebo>
-  -->
+      <gazebo>
+        <plugin name="differential_drive_controller" filename="libgazebo_ros_diff_drive.so">
+          <updateRate>100.0</updateRate>
+          <robotNamespace>/</robotNamespace>
+          <leftJoint>left_wheel_joint</leftJoint>
+          <rightJoint>right_wheel_joint</rightJoint>
+          <wheelSeparation>0.3</wheelSeparation>
+          <wheelDiameter>0.1</wheelDiameter>
+          <robotBaseFrame>base_link</robotBaseFrame>
+          <torque>200</torque>
+          <commandTopic>cmd_vel</commandTopic>
+          <odometryTopic>odom</odometryTopic>
+          <odometryFrame>odom</odometryFrame>
+        </plugin>
+      </gazebo>
+      -->
 </robot>

Commit message: Camera added, but it's a "normal" camera, not an omni.

File: defs/jcf.xacro (robot description, xacro)
@@ -278,11 +278,12 @@
     </plugin>
   </gazebo>
-<!-- test sonar
-  <xacro:sonar_sensor name="s1" parent="base_link"
-    ros_topic="s1" update_rate="10" min_range="0.1" max_range="10"
-    field_of_view="0.267" ray_count="1">
-    <origin xyz="0.2 0 0.22" rpy="0 0 0"/>
-  </xacro:sonar_sensor>
--->
+  <!-- test sonar
+      <xacro:sonar_sensor name="s1" parent="base_link"
+        ros_topic="s1" update_rate="10" min_range="0.1" max_range="10"
+        field_of_view="0.267" ray_count="1">
+        <origin xyz="0.2 0 0.22" rpy="0 0 0"/>
+      </xacro:sonar_sensor>
+      -->
+  <xacro:include filename="$(find gazebo_ros_3dx)/defs/camera.urdf.xacro"/>
   <xacro:include filename="$(find gazebo_ros_3dx)/defs/sonar_pos.urdf.xacro"/>
   <!-- controller

Commit message: Changes to pretty much everything. Now appears to work.

File: defs/jcf.xacro (robot description, xacro)
@@ -27,4 +27,11 @@
   <gazebo reference="base_link">
     <material value="Gazebo/Red"/>
+  </gazebo>
+  <gazebo>
+    <plugin name="lightsensor" filename="liblightsensor_gazebo.so">
+      <link name="base_link"/>
+      <interval>0.1</interval>
+      <pixels>100</pixels>
+    </plugin>
   </gazebo>
   <link name="dummyinertial">
